File: cmvs-rgb.sch (KiCad schematic (older format))
At the start: 14 parts

Commit message: First prototype version
Parts:
- added C2, C3, C4, C5: 220uF, Capacitors_SMD:c_elec_8x10, symbol CP1
- added W1: Jamma_Red, Wire_Pads:SolderWirePad_single_SMD_5x10mm, symbol TEST_1P
- added W10: GND_OUT, Wire_Pads:SolderWirePad_single_SMD_5x10mm, symbol TEST_1P
- added W11: +5V_IN, Wire_Pads:SolderWirePad_single_SMD_5x10mm, symbol TEST_1P
- added W12: +5V_OUT, Wire_Pads:SolderWirePad_single_SMD_5x10mm, symbol TEST_1P
- added W2: Jamma_Blue, Wire_Pads:SolderWirePad_single_SMD_5x10mm, symbol TEST_1P
- added W3: Jamma_Green, Wire_Pads:SolderWirePad_single_SMD_5x10mm, symbol TEST_1P
- added W4: Jamma Sync, Wire_Pads:SolderWirePad_single_SMD_5x10mm, symbol TEST_1P
- added W5: SCART_Red, Wire_Pads:SolderWirePad_single_SMD_5x10mm, symbol TEST_1P
- added W6: SCART_Blue, Wire_Pads:SolderWirePad_single_SMD_5x10mm, symbol TEST_1P
- added W7: SCART_Green, Wire_Pads:SolderWirePad_single_SMD_5x10mm, symbol TEST_1P
- added W8: SCART_Sync, Wire_Pads:SolderWirePad_single_SMD_5x10mm, symbol TEST_1P
- added W9: GND_IN, Wire_Pads:SolderWirePad_single_SMD_5x10mm, symbol TEST_1P
- C1: renamed from C?; footprint (none) -> Capacitors_SMD:C_0603
- R1, R10, R11, R12, R2, R3, R4, R5, R6, R7, R8, R9: renamed from R?; footprint (none) -> Resistors_SMD:R_0603_HandSoldering
- U1: renamed from U?; footprint (none) -> Housings_SSOP:SSOP-14_5.3x6.2mm_Pitch0.65mm
Connections:
- net +5V: now also W11.1, W12.1
- net GND: now also W10.1, W9.1
- net Jamma_Blue: now also W2.1
- net Jamma_Green: now also W3.1
- net Jamma_Red: now also W1.1
- net Jamma_Sync: now also W4.1
- net SCART_Blue: now also C4.2, W7.1; no longer R10.1
- net SCART_Green: now also C3.2, W6.1; no longer R11.1
- net SCART_Red: now also C2.2, W5.1; no longer R9.1
- net SCART_Sync: now also C5.2, W8.1; no longer R12.1
- new net: C2.1, R9.1
- new net: C3.1, R10.1
- new net: C4.1, R11.1
- new net: C5.1, R12.1
Other:
- moved on the sheet: R10, R11, R9

Commit message: V2
* Footprints changed to 0805 for easier soldering
* Solder pads for enabling/disabling LPF
* Corrected voltage divider for Sync signal, Sync toned down to 0.3V
instead of 0.7V
* Smaller PCB
Parts:
- added P1, P2: CONN_01X02, Solderpads:SOLDER-JUMPER_1-WAY, symbol CONN_01X02
- C1: footprint Capacitors_SMD:C_0603 -> Capacitors_SMD:C_0805_HandSoldering
- R1, R10, R11, R12, R2, R3, R4, R6, R7, R8, R9: footprint Resistors_SMD:R_0603_HandSoldering -> Resistors_SMD:R_0805_HandSoldering
- R5: value 1k1 -> 430; footprint Resistors_SMD:R_0603_HandSoldering -> Resistors_SMD:R_0805_HandSoldering
- W1, W10, W11, W12, W2, W3, W4, W5, W6, W7, W8, W9: footprint Wire_Pads:SolderWirePad_single_SMD_5x10mm -> Solderpads:SolderWirePad_single_SMD_3x5mm
Other:
- moved on the sheet: C1
Changed lines of the file:
@@
 F 0 "R7" V 4630 5000 50  0000 C CNN
 F 1 "1k4" V 4550 5000 50  0000 C CNN
-F 2 "Resistors_SMD:R_0603_HandSoldering" V 4480 5000 50  0001 C CNN
+F 2 "Resistors_SMD:R_0805_HandSoldering" V 4480 5000 50  0001 C CNN
 F 3 "" H 4550 5000 50  0000 C CNN
 	1    4550 5000
@@
 F 0 "R6" V 4430 5000 50  0000 C CNN
 F 1 "1k4" V 4350 5000 50  0000 C CNN
-F 2 "Resistors_SMD:R_0603_HandSoldering" V 4280 5000 50  0001 C CNN
+F 2 "Resistors_SMD:R_0805_HandSoldering" V 4280 5000 50  0001 C CNN
 F 3 "" H 4350 5000 50  0000 C CNN
 	1    4350 5000
@@
 P 4150 5000
 F 0 "R5" V 4230 5000 50  0000 C CNN
-F 1 "1k1" V 4150 5000 50  0000 C CNN
-F 2 "Resistors_SMD:R_0603_HandSoldering" V 4080 5000 50  0001 C CNN
+F 1 "430" V 4150 5000 50  0000 C CNN
+F 2 "Resistors_SMD:R_0805_HandSoldering" V 4080 5000 50  0001 C CNN
 F 3 "" H 4150 5000 50  0000 C CNN
 	1    4150 5000
@@
 F 0 "R8" V 4830 5000 50  0000 C CNN
 F 1 "1k4" V 4750 5000 50  0000 C CNN
-F 2 "Resistors_SMD:R_0603_HandSoldering" V 4680 5000 50  0001 C CNN
+F 2 "Resistors_SMD:R_0805_HandSoldering" V 4680 5000 50  0001 C CNN
 F 3 "" H 4750 5000 50  0000 C CNN
 	1    4750 5000
@@
 F 0 "R1" V 3980 4250 50  0000 C CNN
 F 1 "6k8" V 3900 4250 50  0000 C CNN
-F 2 "Resistors_SMD:R_0603_HandSoldering" V 3830 4250 50  0001 C CNN
+F 2 "Resistors_SMD:R_0805_HandSoldering" V 3830 4250 50  0001 C CNN
 F 3 "" H 3900 4250 50  0000 C CNN
 	1    3900 4250
@@
 F 0 "R3" V 3980 4650 50  0000 C CNN
 F 1 "6k8" V 3900 4650 50  0000 C CNN
-F 2 "Resistors_SMD:R_0603_HandSoldering" V 3830 4650 50  0001 C CNN
+F 2 "Resistors_SMD:R_0805_HandSoldering" V 3830 4650 50  0001 C CNN
 F 3 "" H 3900 4650 50  0000 C CNN
 	1    3900 4650
@@
 F 0 "R4" V 3980 4850 50  0000 C CNN
 F 1 "6k8" V 3900 4850 50  0000 C CNN
-F 2 "Resistors_SMD:R_0603_HandSoldering" V 3830 4850 50  0001 C CNN
+F 2 "Resistors_SMD:R_0805_HandSoldering" V 3830 4850 50  0001 C CNN
 F 3 "" H 3900 4850 50  0000 C CNN
 	1    3900 4850
@@
 F 0 "R2" V 3980 4450 50  0000 C CNN
 F 1 "6k8" V 3900 4450 50  0000 C CNN
-F 2 "Resistors_SMD:R_0603_HandSoldering" V 3830 4450 50  0001 C CNN
+F 2 "Resistors_SMD:R_0805_HandSoldering" V 3830 4450 50  0001 C CNN
 F 3 "" H 3900 4450 50  0000 C CNN
 	1    3900 4450
@@
 F 0 "R9" V 7330 3950 50  0000 C CNN
 F 1 "75R" V 7250 3950 50  0000 C CNN
-F 2 "Resistors_SMD:R_0603_HandSoldering" V 7180 3950 50  0001 C CNN
+F 2 "Resistors_SMD:R_0805_HandSoldering" V 7180 3950 50  0001 C CNN
 F 3 "" H 7250 3950 50  0000 C CNN
 	1    7250 3950
@@
 F 0 "R10" V 7330 4250 50  0000 C CNN
 F 1 "75R" V 7250 4250 50  0000 C CNN
-F 2 "Resistors_SMD:R_0603_HandSoldering" V 7180 4250 50  0001 C CNN
+F 2 "Resistors_SMD:R_0805_HandSoldering" V 7180 4250 50  0001 C CNN
 F 3 "" H 7250 4250 50  0000 C CNN
 	1    7250 4250
@@
 F 0 "R11" V 7330 4550 50  0000 C CNN
 F 1 "75R" V 7250 4550 50  0000 C CNN
-F 2 "Resistors_SMD:R_0603_HandSoldering" V 7180 4550 50  0001 C CNN
+F 2 "Resistors_SMD:R_0805_HandSoldering" V 7180 4550 50  0001 C CNN
 F 3 "" H 7250 4550 50  0000 C CNN
 	1    7250 4550
@@
 F 0 "R12" V 7330 4850 50  0000 C CNN
 F 1 "75R" V 7250 4850 50  0000 C CNN
-F 2 "Resistors_SMD:R_0603_HandSoldering" V 7180 4850 50  0001 C CNN
+F 2 "Resistors_SMD:R_0805_HandSoldering" V 7180 4850 50  0001 C CNN
 F 3 "" H 7250 4850 50  0000 C CNN
 	1    7250 4850
@@
 Text GLabel 3500 4250 0    60   Input ~ 0
 Jamma_Red
+Text GLabel 3500 4650 0    60   Input ~ 0
+Jamma_Blue
 Text GLabel 3500 4450 0    60   Input ~ 0
-Jamma_Blue
-Text GLabel 3500 4650 0    60   Input ~ 0
 Jamma_Green
 Text GLabel 3500 4850 0    60   Input ~ 0
@@
 Wire Wire Line
 	6700 5250 6800 5250
-Wire Wire Line
-	6800 5250 6800 5650
-Wire Wire Line
-	4950 5650 7000 5650
-Connection ~ 4950 5650
-$Comp
-L +5V #PWR9
+$Comp
+L +5V #PWR11
 U 1 1 5AC2B239
-P 7000 5050
-F 0 "#PWR9" H 7000 4900 50  0001 C CNN
-F 1 "+5V" H 7000 5190 50  0000 C CNN
-F 2 "" H 7000 5050 50  0000 C CNN
-F 3 "" H 7000 5050 50  0000 C CNN
-	1    7000 5050
+P 7350 5050
+F 0 "#PWR11" H 7350 4900 50  0001 C CNN
+F 1 "+5V" H 7350 5190 50  0000 C CNN
+F 2 "" H 7350 5050 50  0000 C CNN
+F 3 "" H 7350 5050 50  0000 C CNN
+	1    7350 5050
 	1    0    0    -1
 $EndComp
@@
 L C C1
 U 1 1 5AC2B28E
-P 7000 5500
-F 0 "C1" H 7025 5600 50  0000 L CNN
-F 1 "0.1uF" H 7025 5400 50  0000 L CNN
-F 2 "Capacitors_SMD:C_0603" H 7038 5350 50  0001 C CNN
-F 3 "" H 7000 5500 50  0000 C CNN
-	1    7000 5500
-	1    0    0    -1
-$EndComp
-Wire Wire Line
-	6700 5050 7000 5050
-Wire Wire Line
-	7000 5050 7000 5350
-Connection ~ 6800 5650
+P 7350 5200
+F 0 "C1" H 7375 5300 50  0000 L CNN
+F 1 "0.1uF" H 7375 5100 50  0000 L CNN
+F 2 "Capacitors_SMD:C_0805_HandSoldering" H 7388 5050 50  0001 C CNN
+F 3 "" H 7350 5200 50  0000 C CNN
+	1    7350 5200
+	1    0    0    -1
+$EndComp
+Wire Wire Line
+	6700 5050 7350 5050
 $Comp
 L CP1 C2
@@
 F 0 "W1" V 2900 3200 50  0000 C CNN
 F 1 "Jamma_Red" V 3000 3450 50  0000 C CNN
-F 2 "Wire_Pads:SolderWirePad_single_SMD_5x10mm" V 3200 3050 50  0001 C CNN
+F 2 "Solderpads:SolderWirePad_single_SMD_3x5mm" V 3200 3050 50  0001 C CNN
 F 3 "" H 3200 3050 50  0000 C CNN
 	1    3000 3050
@@
 F 0 "W4" V 2900 3800 50  0000 C CNN
 F 1 "Jamma Sync" V 3000 4050 50  0000 C CNN
-F 2 "Wire_Pads:SolderWirePad_single_SMD_5x10mm" H 3200 3650 50  0001 C CNN
+F 2 "Solderpads:SolderWirePad_single_SMD_3x5mm" H 3200 3650 50  0001 C CNN
 F 3 "" H 3200 3650 50  0000 C CNN
 	1    3000 3650
@@
 F 0 "W3" V 2900 3600 50  0000 C CNN
 F 1 "Jamma_Green" V 3000 3900 50  0000 C CNN
-F 2 "Wire_Pads:SolderWirePad_single_SMD_5x10mm" H 3200 3450 50  0001 C CNN
+F 2 "Solderpads:SolderWirePad_single_SMD_3x5mm" H 3200 3450 50  0001 C CNN
 F 3 "" H 3200 3450 50  0000 C CNN
 	1    3000 3450
@@
 F 0 "W2" V 2900 3400 50  0000 C CNN
 F 1 "Jamma_Blue" V 3000 3650 50  0000 C CNN
-F 2 "Wire_Pads:SolderWirePad_single_SMD_5x10mm" H 3200 3250 50  0001 C CNN
+F 2 "Solderpads:SolderWirePad_single_SMD_3x5mm" H 3200 3250 50  0001 C CNN
 F 3 "" H 3200 3250 50  0000 C CNN
 	1    3000 3250
@@
 F 0 "W5" V 5700 3200 50  0000 C CNN
 F 1 "SCART_Red" V 5800 3450 50  0000 C CNN
-F 2 "Wire_Pads:SolderWirePad_single_SMD_5x10mm" V 6000 3050 50  0001 C CNN
+F 2 "Solderpads:SolderWirePad_single_SMD_3x5mm" V 6000 3050 50  0001 C CNN
 F 3 "" H 6000 3050 50  0000 C CNN
 	1    5800 3050
@@
 F 0 "W6" V 5700 3400 50  0000 C CNN
 F 1 "SCART_Blue" V 5800 3650 50  0000 C CNN
-F 2 "Wire_Pads:SolderWirePad_single_SMD_5x10mm" H 6000 3250 50  0001 C CNN
+F 2 "Solderpads:SolderWirePad_single_SMD_3x5mm" H 6000 3250 50  0001 C CNN
 F 3 "" H 6000 3250 50  0000 C CNN
 	1    5800 3250
@@
 F 0 "W7" V 5700 3600 50  0000 C CNN
 F 1 "SCART_Green" V 5800 3900 50  0000 C CNN
-F 2 "Wire_Pads:SolderWirePad_single_SMD_5x10mm" H 6000 3450 50  0001 C CNN
+F 2 "Solderpads:SolderWirePad_single_SMD_3x5mm" H 6000 3450 50  0001 C CNN
 F 3 "" H 6000 3450 50  0000 C CNN
 	1    5800 3450
@@
 F 0 "W8" V 5700 3800 50  0000 C CNN
 F 1 "SCART_Sync" V 5800 4050 50  0000 C CNN
-F 2 "Wire_Pads:SolderWirePad_single_SMD_5x10mm" H 6000 3650 50  0001 C CNN
+F 2 "Solderpads:SolderWirePad_single_SMD_3x5mm" H 6000 3650 50  0001 C CNN
 F 3 "" H 6000 3650 50  0000 C CNN
 	1    5800 3650
@@
 F 0 "W9" H 3150 1670 50  0000 C CNN
 F 1 "GND_IN" H 3150 1600 50  0000 C CNN
-F 2 "Wire_Pads:SolderWirePad_single_SMD_5x10mm" H 3350 1400 50  0001 C CNN
+F 2 "Solderpads:SolderWirePad_single_SMD_3x5mm" H 3350 1400 50  0001 C CNN
 F 3 "" H 3350 1400 50  0000 C CNN
 	1    3150 1400
@@
 F 0 "W10" H 3700 1670 50  0000 C CNN
 F 1 "GND_OUT" H 3700 1600 50  0000 C CNN
-F 2 "Wire_Pads:SolderWirePad_single_SMD_5x10mm" H 3900 1400 50  0001 C CNN
+F 2 "Solderpads:SolderWirePad_single_SMD_3x5mm" H 3900 1400 50  0001 C CNN
 F 3 "" H 3900 1400 50  0000 C CNN
 	1    3700 1400
@@
 F 0 "W11" H 4200 1670 50  0000 C CNN
 F 1 "+5V_IN" H 4200 1600 50  0000 C CNN
-F 2 "Wire_Pads:SolderWirePad_single_SMD_5x10mm" H 4400 1400 50  0001 C CNN
+F 2 "Solderpads:SolderWirePad_single_SMD_3x5mm" H 4400 1400 50  0001 C CNN
 F 3 "" H 4400 1400 50  0000 C CNN
 	1    4200 1400
@@
 F 0 "W12" H 4650 1670 50  0000 C CNN
 F 1 "+5V_OUT" H 4650 1600 50  0000 C CNN
-F 2 "Wire_Pads:SolderWirePad_single_SMD_5x10mm" H 4850 1400 50  0001 C CNN
+F 2 "Solderpads:SolderWirePad_single_SMD_3x5mm" H 4850 1400 50  0001 C CNN
 F 3 "" H 4850 1400 50  0000 C CNN
 	1    4650 1400
@@
 	1    0    0    -1
 $EndComp
+$Comp
+L GND #PWR12
+U 1 1 5AD46286
+P 7350 5350
+F 0 "#PWR12" H 7350 5100 50  0001 C CNN
+F 1 "GND" H 7350 5200 50  0000 C CNN
+F 2 "" H 7350 5350 50  0001 C CNN
+F 3 "" H 7350 5350 50  0001 C CNN
+	1    7350 5350
+	1    0    0    -1
+$EndComp
+$Comp
+L GND #PWR10
+U 1 1 5AD46E15
+P 7100 6200
+F 0 "#PWR10" H 7100 5950 50  0001 C CNN
+F 1 "GND" H 7100 6050 50  0000 C CNN
+F 2 "" H 7100 6200 50  0001 C CNN
+F 3 "" H 7100 6200 50  0001 C CNN
+	1    7100 6200
+	1    0    0    -1
+$EndComp
+$Comp
+L +5V #PWR9
+U 1 1 5AD46EE6
+P 7100 5750
+F 0 "#PWR9" H 7100 5600 50  0001 C CNN
+F 1 "+5V" H 7100 5890 50  0000 C CNN
+F 2 "" H 7100 5750 50  0001 C CNN
+F 3 "" H 7100 5750 50  0001 C CNN
+	1    7100 5750
+	1    0    0    -1
+$EndComp
+Wire Wire Line
+	6800 5250 6800 5850
+Wire Wire Line
+	6800 5850 7100 5850
+$Comp
+L CONN_01X02 P1
+U 1 1 5B0C0BF6
+P 7300 5800
+F 0 "P1" H 7300 5950 50  0000 C CNN
+F 1 "CONN_01X02" V 7400 5800 50  0000 C CNN
+F 2 "Solderpads:SOLDER-JUMPER_1-WAY" H 7300 5800 50  0001 C CNN
+F 3 "" H 7300 5800 50  0000 C CNN
+	1    7300 5800
+	1    0    0    -1
+$EndComp
+$Comp
+L CONN_01X02 P2
+U 1 1 5B0C0C7D
+P 7300 6150
+F 0 "P2" H 7300 6300 50  0000 C CNN
+F 1 "CONN_01X02" V 7400 6150 50  0000 C CNN
+F 2 "Solderpads:SOLDER-JUMPER_1-WAY" H 7300 6150 50  0001 C CNN
+F 3 "" H 7300 6150 50  0000 C CNN
+	1    7300 6150
+	1    0    0    -1
+$EndComp
+Wire Wire Line
+	7100 5850 7100 6100
 $EndSCHEMATC
